File: kicad_docs/CEM3340_VCO.kicad_pcb (KiCad board)
At the start: 2 copper layers, 55.9 x 78.7 mm, 96 parts, among them J1 tuning controls, J2 1 v/oct inputs, J3 linear FM input, J4 sync input, J5 PWM inputs, J6 power input, Q1 MMDT3904, U1 L78L10_SOT89, U2 MC7905, U3 REF02AU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

Commit message: place github url on pcb silk
Other:
- board text added: "github.com/JordanAceto/CEM3340_VCO rev 0 01/29/2020"
Changed lines of the file:
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@@
   (general
     (thickness 1.6)
-    (drawings 59)
+    (drawings 60)
     (tracks 592)
     (zones 0)
@@
     (34 B.Paste user)
     (35 F.Paste user)
-    (36 B.SilkS user hide)
+    (36 B.SilkS user)
     (37 F.SilkS user)
     (38 B.Mask user)
@@
   )
   (setup
-    (last_trace_width 0.4)
+    (last_trace_width 0.25)
     (user_trace_width 0.4)
     (trace_clearance 0.2)
@@
     )
   )
+  (gr_text "github.com/JordanAceto/CEM3340_VCO\nrev 0\n01/29/2020" (at 130.81 54.61) (layer B.SilkS)
+    (effects (font (size 1 1) (thickness 0.15)) (justify left mirror))
+  )
   (gr_text j6 (at 82.55 76.2) (layer B.SilkS)
