File: kicad_docs/VCO_Core.sch (KiCad schematic (older format))
At the start: 26 parts, among them U4 CEM3340

Commit message: update and fill in some resistor values
Other:
- note added: "about 3.4 vpp"
- note added: "about 6.8 vpp"
- note removed: "about ???vpp"
Changed lines of the file:
@@
 encoding utf-8
 Sheet 4 4
-Title ""
+Title "CEM3340 VCO Core"
 Date "2020-01-30"
 Rev "1"
@@
 	6200 5200 6200 5350
 Text Notes 5850 2900 0    59   ~ 0
-about ???vpp
+about 3.4 vpp
 Text Notes 4350 3400 0    59   ~ 0
-about ???vpp
-$Comp
-L Device:R R?
+about 6.8 vpp
+$Comp
+L Device:R R?
