File: kicad_docs/Waveshapers.sch (KiCad schematic (older format))
At the start: 30 parts, among them Q1 MMDT3904, U5 TL072, U6 TL072, U7 TL072

Commit message: update and fill in some resistor values
Parts:
- R30: value ??? -> 34k
- R32: value ??? -> 68k
Other:
- note added: "choose r40 and r44 to get a \n10 vpp pulse wave with an\noutput impedance of around 1k ohm"
Changed lines of the file:
@@
 encoding utf-8
 Sheet 3 4
-Title ""
+Title "CEM3340 VCO Waveshapers"
 Date "2020-01-30"
 Rev "1"
@@
 AR Path="/5E3EF2A7/5E7D17BF" Ref="R30"  Part="1"
 F 0 "R30" V 2200 1400 50  0000 C CNN
-F 1 "???" V 2300 1400 50  0000 C CNN
+F 1 "34k" V 2300 1400 50  0000 C CNN
 F 2 "Resistor_SMD:R_0805_2012Metric_Pad1.15x1.40mm_HandSolder" V 2230 1400 50  0001 C CNN
 F 3 "~" H 2300 1400 50  0001 C CNN
@@
 AR Path="/5E3EF2A7/5E7D17E2" Ref="R32"  Part="1"
 F 0 "R32" V 2200 3550 50  0000 C CNN
-F 1 "???" V 2300 3550 50  0000 C CNN
+F 1 "68k" V 2300 3550 50  0000 C CNN
 F 2 "Resistor_SMD:R_0805_2012Metric_Pad1.15x1.40mm_HandSolder" V 2230 3550 50  0001 C CNN
 F 3 "~" H 2300 3550 50  0001 C CNN
@@
 Wire Wire Line
 	3750 4050 3650 4050
+Text Notes 4100 6200 0    59   ~ 0
+choose r40 and r44 to get a \n10 vpp pulse wave with an\noutput impedance of around 1k ohm
 $EndSCHEMATC

Commit message: increase sine level to 10vpp
Parts:
- R35, R36: value 11k -> 15k
Changed lines of the file:
@@
 AR Path="/5E3EF2A7/5E7D16B2" Ref="R36"  Part="1"
 F 0 "R36" V 9150 1650 50  0000 C CNN
-F 1 "11k" V 9250 1650 50  0000 C CNN
+F 1 "15k" V 9250 1650 50  0000 C CNN
 F 2 "Resistor_SMD:R_0805_2012Metric_Pad1.15x1.40mm_HandSolder" V 9180 1650 50  0001 C CNN
 F 3 "~" H 9250 1650 50  0001 C CNN
@@
 AR Path="/5E3EF2A7/5E7D16CA" Ref="R35"  Part="1"
 F 0 "R35" H 8730 2454 50  0000 R CNN
-F 1 "11k" V 8800 2550 50  0000 R CNN
+F 1 "15k" V 8800 2550 50  0000 R CNN
 F 2 "Resistor_SMD:R_0805_2012Metric_Pad1.15x1.40mm_HandSolder" V 8730 2500 50  0001 C CNN
 F 3 "~" H 8800 2500 50  0001 C CNN

Commit message: finalize some values, update documentation
Parts:
- R40, R44: value R -> 2k
Changed lines of the file:
@@
 AR Path="/5E3EF2A7/5E7D1784" Ref="R40"  Part="1"
 F 0 "R40" V 3800 6300 50  0000 C CNN
-F 1 "R" V 3900 6300 50  0000 C CNN
+F 1 "2k" V 3900 6300 50  0000 C CNN
 F 2 "Resistor_SMD:R_0805_2012Metric_Pad1.15x1.40mm_HandSolder" V 3830 6300 50  0001 C CNN
 F 3 "~" H 3900 6300 50  0001 C CNN
@@
 AR Path="/5E3EF2A7/5E7D1798" Ref="R44"  Part="1"
 F 0 "R44" H 4350 6650 50  0000 L CNN
-F 1 "R" V 4300 6650 50  0000 L CNN
+F 1 "2k" V 4300 6650 50  0000 L CNN
 F 2 "Resistor_SMD:R_0805_2012Metric_Pad1.15x1.40mm_HandSolder" V 4230 6650 50  0001 C CNN
 F 3 "~" H 4300 6650 50  0001 C CNN
